File: pico-probe.kicad_pcb (KiCad board)
At the start: 2 copper layers, 36 parts, among them J1 Conn_01x04, J2 USB_C_Receptacle_USB2.0, J3 Conn_01x05, SW1 SW_Push, U1 RP2040, U3 USBLC6-4SC6, U4 SPX1117-3.3, U5 W25Q16JVSS, Y1 Crystal_GND24

Commit message: 布线
Parts:
- added D2: ESD5341, KisonNew:esd5341, F.Cu at (146.6, 124.2)
- added D5: ESD5341, KisonNew:esd5341, F.Cu at (146.6, 127.0)
- moved R4 4.63 mm to (146.0, 140.1), turned to 0 degrees
- moved C15 3.17 mm to (129.9, 141.7), turned to 180 degrees
- moved J1 2.89 mm to (150.1, 123.4)
- moved D3 2.68 mm to (146.1, 128.6)
- moved C14 2.61 mm to (138.8, 140.2), turned to 180 degrees
- moved C6 2.45 mm to (142.6, 125.4)
- moved D4 2.39 mm to (145.8, 130.1)
- moved C1 2.04 mm to (132.4, 135.5)
- moved C2 2.04 mm to (136.9, 135.4)
- moved R1 2.04 mm to (134.6, 135.5)
- moved R2 2.04 mm to (133.5, 135.5)
- moved C11 2.04 mm to (135.8, 135.5)
- moved D1 2.03 mm to (129.9, 137.4)
- moved U3 1.92 mm to (134.6, 138.6), turned to 0 degrees
- moved C4 1.65 mm to (145.1, 131.2)
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Connections:
- JP1 pad 3: /EXT_5V -> +5V
Routing:
- net +3V3: track 0.00 -> 132.9 mm, vias 0 -> 4
- net VBUS: track 0.00 -> 63.8 mm, vias 0 -> 2
- net /DeviceVcc: track 0.00 -> 30.6 mm
- net /GPIO2: track 0.00 -> 23.9 mm, vias 0 -> 1
- net /GPIO3: track 0.00 -> 23.0 mm, vias 0 -> 1
- net +1V1: track 0.00 -> 21.3 mm
- net /USB_D-: track 0.00 -> 18.8 mm
- net /QSPI_SS: track 0.00 -> 15.3 mm, vias 0 -> 2
- net /QSPI_SD1: track 0.00 -> 14.8 mm, vias 0 -> 2
- net /USB_D+: track 0.00 -> 14.3 mm
- net GND: track 0.00 -> 14.1 mm, vias 0 -> 11
- net Net-(J2-PadA5): track 0.00 -> 13.0 mm, vias 0 -> 2
- net /GPIO5: track 0.00 -> 11.4 mm
- net /GPIO4: track 0.00 -> 11.2 mm
- net /QSPI_SD2: track 0.00 -> 10.9 mm
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- added copper zone on B.Cu, net GND
- added copper zone on F.Cu, net GND
Other:
- board outline added: 37 x 37 mm

Commit message: 新布线
Parts:
- C15, C16: footprint Capacitor_SMD:C_0805_2012Metric -> Capacitor_SMD:C_0603_1608Metric
Connections:
- J3 pad 1: unconnected-(J3-Pad1) -> /DeviceVcc
Routing:
- net GND: track 14.1 -> 108.3 mm, vias 11 -> 25
- net /DeviceVcc: track 30.6 -> 54.8 mm
- net +3V3: track 132.9 -> 134.6 mm
- net VBUS: track 63.8 -> 65.1 mm
- added copper zone on F.Cu, net +1V1
- added copper zone on F.Cu, net +3V3
Other:
- board text added: "CLK"
- board text added: "DIO"
- board text added: "GND"
- board text added: "NC"
- board text added: "VCC"

Commit message: 添加LED
Parts:
- added D6: LEDW, LED_SMD:LED_0603_1608Metric, F.Cu at (128.2, 128.8)
- added R8: 10k, Resistor_SMD:R_0402_1005Metric, F.Cu at (125.1, 125.2)
Routing:
- net /GPIO25: track 0.00 -> 7.44 mm, vias 0 -> 2
- net Net-(D6-Pad1): track 0.00 -> 4.04 mm
Changed lines of the file:
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@@
   (net 59 "unconnected-(J3-Pad5)")
   (net 60 "unconnected-(U3-Pad3)")
+  (net 61 "Net-(D6-Pad1)")
   (footprint "KisonNew:C9002" (layer "F.Cu")
     (at 136.071947 121.424118)
@@
     (tags "esd")
     (property "LCSC" "C239773")
-    (property "Price" "0.2")
+    (property "Price" "")
     (property "Sheetfile" "pico-probe.kicad_sch")
     (property "Sheetname" "")
@@
     (tags "esd")
     (property "LCSC" "C239773")
-    (property "Price" "0.2")
+    (property "Price" "")
     (property "Sheetfile" "pico-probe.kicad_sch")
     (property "Sheetname" "")
@@
       (net 18 "VBUS") (pinfunction "A") (pintype "passive"))
   )
+  (footprint "Resistor_SMD:R_0402_1005Metric" (layer "F.Cu")
+    (at 125.08 125.23 -90)
+    (descr "Resistor SMD 0402 (1005 Metric), square (rectangular) end terminal, IPC_7351 nominal, (Body size source: IPC-SM-782 page 72, https://www.pcb-3d.com/wordpress/wp-content/uploads/ipc-sm-782a_amendment_1_and_2.pdf), generated with kicad-footprint-generator")
+    (tags "resistor")
+    (property "LCSC" "C25744")
+    (property "Price" "")
+    (property "Sheetfile" "pico-probe.kicad_sch")
+    (property "Sheetname" "")
+    (attr smd)
+    (fp_text reference "R8" (at 0 -1.17 90) (layer "F.SilkS") hide
+      (effects (font (size 1 1) (thickness 0.15)))
+    )
+    (fp_text value "10k" (at 0 1.17 90) (layer "F.Fab")
+      (effects (font (size 1 1) (thickness 0.15)))
+    )
+    (fp_text user "${REFERENCE}" (at 0 0 90) (layer "F.Fab")
+      (effects (font (size 0.26 0.26) (thickness 0.04)))
+    )
+    (fp_line (start -0.153641 0.38) (end 0.153641 0.38) (layer "F.SilkS") (width 0.12))
+    (fp_line (start -0.153641 -0.38) (end 0.153641 -0.38) (layer "F.SilkS") (width 0.12))
+    (fp_line (start 0.93 -0.47) (end 0.93 0.47) (layer "F.CrtYd") (width 0.05))
+    (fp_line (start 0.93 0.47) (end -0.93 0.47) (layer "F.CrtYd") (width 0.05))
+    (fp_line (start -0.93 -0.47) (end 0.93 -0.47) (layer "F.CrtYd") (width 0.05))
+    (fp_line (start -0.93 0.47) (end -0.93 -0.47) (layer "F.CrtYd") (width 0.05))
+    (fp_line (start -0.525 0.27) (end -0.525 -0.27) (layer "F.Fab") (width 0.1))
+    (fp_line (start 0.525 0.27) (end -0.525 0.27) (layer "F.Fab") (width 0.1))
+    (fp_line (start 0.525 -0.27) (end 0.525 0.27) (layer "F.Fab") (width 0.1))
+    (fp_line (start -0.525 -0.27) (end 0.525 -0.27) (layer "F.Fab") (width 0.1))
+    (pad "1" smd roundrect (at -0.51 0 270) (size 0.54 0.64) (layers "F.Cu" "F.Paste" "F.Mask") (roundrect_rratio 0.25)
+      (net 2 "GND") (pintype "passive"))
+    (pad "2" smd roundrect (at 0.51 0 270) (size 0.54 0.64) (layers "F.Cu" "F.Paste" "F.Mask") (roundrect_rratio 0.25)
+      (net 61 "Net-(D6-Pad1)") (pintype "passive"))
+    (model "${KICAD6_3DMODEL_DIR}/Resistor_SMD.3dshapes/R_0402_1005Metric.wrl"
+      (offset (xyz 0 0 0))
+      (scale (xyz 1 1 1))
+      (rotate (xyz 0 0 0))
+    )
+  )
   (footprint "Capacitor_SMD:C_0402_1005Metric" (layer "F.Cu")
     (at 136.87 135.45 -90)
@@
     (tags "esd")
     (property "LCSC" "C239773")
-    (property "Price" "0.2")
+    (property "Price" "")
     (property "Sheetfile" "pico-probe.kicad_sch")
     (property "Sheetname" "")
@@
     (tags "capacitor")
     (property "LCSC" "C19702")
-    (property "Price" "0.04")
+    (property "Price" "")
     (property "Sheetfile" "pico-probe.kicad_sch")
     (property "Sheetname" "")
@@
       (net 19 "+5V") (pinfunction "B") (pintype "passive"))
     (model "${KICAD6_3DMODEL_DIR}/Connector_PinHeader_2.54mm.3dshapes/PinHeader_1x03_P2.54mm_Vertical.wrl"
+      (offset (xyz 0 0 0))
+      (scale (xyz 1 1 1))
+      (rotate (xyz 0 0 0))
+    )
+  )
+  (footprint "LED_SMD:LED_0603_1608Metric" (layer "F.Cu")
+    (at 128.15 128.83)
+    (descr "LED SMD 0603 (1608 Metric), square (rectangular) end terminal, IPC_7351 nominal, (Body size source: http://www.tortai-tech.com/upload/download/2011102023233369053.pdf), generated with kicad-footprint-generator")
+    (tags "LED")
+    (property "LCSC" "C2290")
+    (property "Price" "")
+    (property "Sheetfile" "pico-probe.kicad_sch")
+    (property "Sheetname" "")
+    (attr smd)
+    (fp_text reference "D6" (at 0 -1.43) (layer "F.SilkS") hide
+      (effects (font (size 1 1) (thickness 0.15)))
+    )
+    (fp_text value "LEDW" (at 0 1.43) (layer "F.Fab")
+      (effects (font (size 1 1) (thickness 0.15)))
+    )
+    (fp_text user "${REFERENCE}" (at 0 0) (layer "F.Fab")
+      (effects (font (size 0.4 0.4) (thickness 0.06)))
+    )
+    (fp_line (start -1.485 0.735) (end 0.8 0.735) (layer "F.SilkS") (width 0.12))
+    (fp_line (start 0.8 -0.735) (end -1.485 -0.735) (layer "F.SilkS") (width 0.12))
+    (fp_line (start -1.485 -0.735) (end -1.485 0.735) (layer "F.SilkS") (width 0.12))
+    (fp_line (start 1.48 0.73) (end -1.48 0.73) (layer "F.CrtYd") (width 0.05))
+    (fp_line (start -1.48 0.73) (end -1.48 -0.73) (layer "F.CrtYd") (width 0.05))
+    (fp_line (start -1.48 -0.73) (end 1.48 -0.73) (layer "F.CrtYd") (width 0.05))
+    (fp_line (start 1.48 -0.73) (end 1.48 0.73) (layer "F.CrtYd") (width 0.05))
+    (fp_line (start -0.8 0.4) (end 0.8 0.4) (layer "F.Fab") (width 0.1))
+    (fp_line (start -0.5 -0.4) (end -0.8 -0.1) (layer "F.Fab") (width 0.1))
+    (fp_line (start 0.8 -0.4) (end -0.5 -0.4) (layer "F.Fab") (width 0.1))
+    (fp_line (start -0.8 -0.1) (end -0.8 0.4) (layer "F.Fab") (width 0.1))
+    (fp_line (start 0.8 0.4) (end 0.8 -0.4) (layer "F.Fab") (width 0.1))
+    (pad "1" smd roundrect (at -0.7875 0) (size 0.875 0.95) (layers "F.Cu" "F.Paste" "F.Mask") (roundrect_rratio 0.25)
+      (net 61 "Net-(D6-Pad1)") (pinfunction "K") (pintype "passive"))
+    (pad "2" smd roundrect (at 0.7875 0) (size 0.875 0.95) (layers "F.Cu" "F.Paste" "F.Mask") (roundrect_rratio 0.25)
+      (net 54 "/GPIO25") (pinfunction "A") (pintype "passive"))
+    (model "${KICAD6_3DMODEL_DIR}/LED_SMD.3dshapes/LED_0603_1608Metric.wrl"
       (offset (xyz 0 0 0))
       (scale (xyz 1 1 1))
@@
     (tags "esd")
     (property "LCSC" "C239773")
-    (property "Price" "0.2")
+    (property "Price" "")
     (property "Sheetfile" "pico-probe.kicad_sch")
     (property "Sheetname" "")
@@
     (tags "CMS SOT")
     (property "LCSC" "C6862")
-    (property "Price" "0.76")
+    (property "Price" "")
     (property "Sheetfile" "pico-probe.kicad_sch")
     (property "Sheetname" "")
@@
     (tags "capacitor")
     (property "LCSC" "C19702")
-    (property "Price" "0.04")
+    (property "Price" "")
     (property "Sheetfile" "pico-probe.kicad_sch")
     (property "Sheetname" "")
@@
   (segment (start 141.83 128.91) (end 146.05 124.69) (width 0.2) (layer "F.Cu") (net 31))
   (segment (start 140.96 128.91) (end 141.83 128.91) (width 0.2) (layer "F.Cu") (net 31))
+  (segment (start 128.9375 128.83) (end 128.9375 127.4325) (width 0.2) (layer "F.Cu") (net 54))
+  (segment (start 134.085 129.31) (end 132.56 129.31) (width 0.2) (layer "F.Cu") (net 54))
+  (segment (start 132.56 129.31) (end 132.43 129.18) (width 0.2) (layer "F.Cu") (net 54))
+  (segment (start 128.9375 127.4325) (end 129.08 127.29) (width 0.2) (layer "F.Cu") (net 54))
+  (via (at 129.08 127.29) (size 0.8) (drill 0.4) (layers "F.Cu" "B.Cu") (net 54))
+  (via (at 132.43 129.18) (size 0.8) (drill 0.4) (layers "F.Cu" "B.Cu") (net 54))
+  (segment (start 130.97 129.18) (end 129.08 127.29) (width 0.2) (layer "B.Cu") (net 54))
+  (segment (start 132.43 129.18) (end 130.97 129.18) (width 0.2) (layer "B.Cu") (net 54))
+  (segment (start 127.3625 128.0225) (end 125.08 125.74) (width 0.2) (layer "F.Cu") (net 61))
+  (segment (start 127.3625 128.83) (end 127.3625 128.0225) (width 0.2) (layer "F.Cu") (net 61))
   (zone (net 3) (net_name "+3V3") (layer "F.Cu") (hatch edge 0.508)
     (connect_pads (clearance 0.508))
